File: snk75/_autosave-snk75.kicad_pcb (KiCad board)
At the start: 2 copper layers, 274 parts, among them J1 USB_C_Receptacle_USB2.0, U1 ATmega32U4-AU, Y1 16MHZ

Commit message: Switch layout on PCB Editor
Parts:
- moved R12 471.7 mm to (66.7, 174.4)
- moved R16 471.7 mm to (66.7, 181.0)
- moved R20 471.7 mm to (72.6, 177.7)
- moved R23 471.7 mm to (72.6, 184.3)
- moved R27 471.7 mm to (66.7, 177.7)
- moved R54 471.7 mm to (66.7, 167.8)
- moved R56 471.7 mm to (72.6, 181.0)
- moved R76 471.7 mm to (66.7, 171.1)
- moved R81 471.7 mm to (72.6, 167.8)
- moved R87 471.7 mm to (72.6, 174.4)
- moved R9 471.7 mm to (72.6, 171.1)
- moved R10 410.7 mm to (29.8, 181.3)
- moved R13 410.7 mm to (29.8, 174.7)
- moved R15 410.7 mm to (23.8, 178.0)
- moved R24 410.7 mm to (29.8, 168.2)
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