File: snk75/components.kicad_sch (KiCad schematic)
At the start: 10 parts, among them Q1 AO3400A

Commit message: added new row layout and connected row1 to MCU
Parts:
- added C28, C29: 100uF, Capacitor_Tantalum_SMD:CP_EIA-3528-21_Kemet-B, symbol Device:C_Small
- added C30: 10uF, Capacitor_Tantalum_SMD:CP_EIA-3216-18_Kemet-A, symbol Device:C_Small
- added C31, C34: 1uF, Capacitor_SMD:C_0402_1005Metric, symbol Device:C_Small
- added C32, C39, C41: 4.7uF, Capacitor_SMD:C_0402_1005Metric, symbol Device:C_Small
- added C35, C36, C37, C38: 100nF, Capacitor_SMD:C_0402_1005Metric, symbol Device:C_Small
- added C40, C43: 1u, Capacitor_SMD:C_0805_2012Metric, symbol Device:C
- added C42: 10n, Capacitor_SMD:C_0402_1005Metric, symbol Device:C_Small
- added D102: B5819W-SL, acheron_Components:D_SOD-123, symbol Device:D_Schottky
- added F1: nSMD100-16V, Fuse:Fuse_1206_3216Metric, symbol Device:Fuse
- added F2: 500m, Fuse:Fuse_1206_3216Metric, symbol Device:Polyfuse_Small
- added J2: USB_C_Receptacle_USB2.0, Connector_USB:USB_C_Receptacle_HRO_TYPE-C-31-M-12, symbol Connector:USB_C_Receptacle_USB2.0
- added R108: 0, Resistor_SMD:R_0402_1005Metric, symbol Device:R_Small
- added R109: 100k, Resistor_SMD:R_0402_1005Metric, symbol Device:R
- added R110, R111: 5.1k, Resistor_SMD:R_0402_1005Metric, symbol Device:R_Small
- added R112: 100k, Resistor_SMD:R_0805_2012Metric, symbol Device:R
- added U3: USBLC6-2SC6, Package_TO_SOT_SMD:SOT-23-6_Handsoldering, symbol Power_Protection:USBLC6-2SC6
- added U4: XC6206P332MR, Package_TO_SOT_SMD:SOT-23_Handsoldering, symbol isometria-75-pcb-iso-rescue:XC6206PxxxMR-Regulator_Linear-kicad-keyboard-parts
- added U5: SGM2007-3.3XN5/TR, Package_TO_SOT_SMD:SOT-23-5_HandSoldering, symbol acheron_Symbols:SGM2036
- C33: renamed from C29; footprint (none) -> Capacitor_SMD:C_0402_1005Metric
- R107: renamed from R93; footprint (none) -> Resistor_SMD:R_0402_1005Metric
- renumbered C28 to C27, R89 to R103, R90 to R104, R91 to R105, R92 to R106
Connections:
- net +3V3: now also C34.1, C35.1, C36.1, C37.1, C38.1, C39.1, C41.1, U4.2 (VO)
- net +5V: now also C28.1, C29.1, C30.1, C31.1, C32.1, U4.3 (VI)
- net GND: now also C28.2, C29.2, C30.2, C31.2, C32.2, C34.2, C35.2, C36.2, C37.2, C38.2, C39.2, C40.2, C41.2, C42.1, C43.1, J2.S1 (SHIELD), R108.2, R109.2, R112.1, U3.2 (GND), U4.1 (GND), U5.2 (GND)
- new net: J2.A5 (CC1), R110.2
- new net: C42.2, U5.4 (BP/FB)
- new net: F2.1, J2.A4 (VBUS), J2.A9 (VBUS), J2.B4 (VBUS), J2.B9 (VBUS)
- new net: J2.A1 (GND), J2.A12 (GND), J2.B1 (GND), J2.B12 (GND), R108.1
- new net: J2.B5 (CC2), R111.2
- new net 3V3: C43.2, D102.2 (A), R112.2, U5.5 (OUT)
- new net 5V: C40.1, D102.1 (K), F1.1, R109.1, U5.1 (IN), U5.3 (EN)
- new net D+: J2.A6 (D+), J2.B6 (D+), U3.1 (I/O1)
- new net D-: J2.A7 (D-), J2.B7 (D-), U3.3 (I/O2)
- new net DBUS+: U3.6 (I/O1)
- new net DBUS-: U3.4 (I/O2)
- new net GNDPWR: R110.1, R111.1
- new net VOUT: F1.2, F2.2, U3.5 (VBUS)
- no-connect marks 0 -> 2
Other:
- note added: "3V3"
- note added: "BOOT"
- note added: "USB-C ESD (Suppressor)"
- note added: "USBC Receptacle"
- note added: "Voltage regulation + filtering"
