File: snk75/snk75.kicad_pcb (KiCad board)
At the start: 2 copper layers, 314.3 x 123.8 mm, 313 parts, among them J1 TYPE-C-31-M12_13, Q1 AO3400A, U1 ATmega32U4-AU, U2 USBLC6-2SC6, U3 74LVC1G125, Y1 16MHZ

Commit message: added new row layout and connected row1 to MCU
Parts:
- removed C1: 22pF, Capacitor_SMD:C_0402_1005Metric
- removed C2: 22pF, Capacitor_SMD:C_0402_1005Metric_Pad0.74x0.62mm_HandSolder
- removed C3: 1u, Capacitor_SMD:C_0402_1005Metric_Pad0.74x0.62mm_HandSolder
- removed C4: 100nF, Capacitor_SMD:C_0402_1005Metric_Pad0.74x0.62mm_HandSolder
- removed C5: 10u, Capacitor_SMD:C_0402_1005Metric
- removed C6, C9: 1u, Capacitor_SMD:C_0402_1005Metric
- removed C7, C8: 100n, Capacitor_SMD:C_0402_1005Metric
- removed FB1: FerriteBead_Small, Inductor_SMD:L_0805_2012Metric
- removed J1: TYPE-C-31-M12_13, acheron_Connectors:TYPE-C-31-M-12
- removed R1: 10k, Resistor_SMD:R_0402_1005Metric
- removed U1: ATmega32U4-AU, Package_QFP:TQFP-44_10x10mm_P0.8mm
- removed Y1: 16MHZ, Crystal:Crystal_SMD_5032-2Pin_5.0x3.2mm_HandSoldering
- added C28: 100uF, Capacitor_Tantalum_SMD:CP_EIA-3528-21_Kemet-B, B.Cu at (-29.8, 21.5)
- added C29: 100uF, Capacitor_Tantalum_SMD:CP_EIA-3528-21_Kemet-B, B.Cu at (-41.4, 14.6)
- added C30: 10uF, Capacitor_Tantalum_SMD:CP_EIA-3216-18_Kemet-A, B.Cu at (-35.6, 20.9)
- added C31: 1uF, Capacitor_SMD:C_0402_1005Metric, B.Cu at (-51.4, 14.3)
- added C32: 4.7uF, Capacitor_SMD:C_0402_1005Metric, B.Cu at (-50.3, 18.7)
- added C33: 100nF, Capacitor_SMD:C_0402_1005Metric, B.Cu at (-64.6, 3.66)
- added C34: 1uF, Capacitor_SMD:C_0402_1005Metric, B.Cu at (-50.3, 16.7)
- added C35: 100nF, Capacitor_SMD:C_0402_1005Metric, B.Cu at (-54.3, 12.3)
- added C36: 100nF, Capacitor_SMD:C_0402_1005Metric, B.Cu at (-47.2, 21.7)
- added C37: 100nF, Capacitor_SMD:C_0402_1005Metric, B.Cu at (-59.5, 8.11)
- added C38: 100nF, Capacitor_SMD:C_0402_1005Metric, B.Cu at (-42.9, 23.7)
- added C39: 4.7uF, Capacitor_SMD:C_0402_1005Metric, B.Cu at (-47.2, 19.7)
- added C40: 1u, Capacitor_SMD:C_0805_2012Metric, B.Cu at (-40.7, 18.3)
- added C41: 4.7uF, Capacitor_SMD:C_0402_1005Metric, B.Cu at (-56.8, 10.1)
- added C42: 10n, Capacitor_SMD:C_0402_1005Metric, B.Cu at (-61.7, 5.65)
- added C43: 1u, Capacitor_SMD:C_0805_2012Metric, B.Cu at (-46.6, 17.2)
- added D102: B5819W-SL, acheron_Components:D_SOD-123, B.Cu at (-52.5, 4.35)
- added F1: nSMD100-16V, Fuse:Fuse_1206_3216Metric, B.Cu at (-47.2, 14.1)
- added F2: 500m, Fuse:Fuse_1206_3216Metric, B.Cu at (-52.3, 7.67)
- added J2: USB_C_Receptacle_USB2.0, Connector_USB:USB_C_Receptacle_HRO_TYPE-C-31-M-12, B.Cu at (14.0, 26.2)
- added R100: 5.1R, Resistor_SMD:R_0402_1005Metric, B.Cu at (-76.4, 3.67)
- added R101: 5.1R, Resistor_SMD:R_0402_1005Metric, B.Cu at (-70.5, 11.6)
- added R102: 5.1R, Resistor_SMD:R_0402_1005Metric, B.Cu at (-73.5, 3.67)
- added R103: 330, Resistor_SMD:R_0402_1005Metric, B.Cu at (-40.0, 23.7)
- added R104: 10k, Resistor_SMD:R_0402_1005Metric, B.Cu at (-37.1, 23.7)
- added R105: 10k, Resistor_SMD:R_0402_1005Metric, B.Cu at (-51.0, 10.3)
- added R106: 100R, Resistor_SMD:R_0402_1005Metric, B.Cu at (-34.2, 23.5)
- added R107: 10k, Resistor_SMD:R_0402_1005Metric, B.Cu at (-53.9, 10.3)
- added R108: 0, Resistor_SMD:R_0402_1005Metric, B.Cu at (-44.3, 20.8)
- added R109: 100k, Resistor_SMD:R_0402_1005Metric, B.Cu at (-61.7, 3.67)
- added R110: 5.1k, Resistor_SMD:R_0402_1005Metric, B.Cu at (-51.5, 12.3)
- added R111: 5.1k, Resistor_SMD:R_0402_1005Metric, B.Cu at (-56.6, 8.12)
- added R112: 100k, Resistor_SMD:R_0805_2012Metric, B.Cu at (-40.6, 21.2)
- added R93: 5.1R, Resistor_SMD:R_0402_1005Metric, B.Cu at (-73.5, 5.66)
- added R94: 5.1R, Resistor_SMD:R_0402_1005Metric, B.Cu at (-76.4, 5.66)
- added R95: 5.1R, Resistor_SMD:R_0402_1005Metric, B.Cu at (-70.5, 5.66)
- added R96: 5.1R, Resistor_SMD:R_0402_1005Metric, B.Cu at (-70.5, 3.67)
- added R97: 5.1R, Resistor_SMD:R_0402_1005Metric, B.Cu at (-70.5, 7.65)
- added R98: 5.1R, Resistor_SMD:R_0402_1005Metric, B.Cu at (-73.5, 7.65)
- added R99: 5.1R, Resistor_SMD:R_0402_1005Metric, B.Cu at (-70.5, 9.64)
- added SWP2: SW_Push_BOOT, Button_Switch_SMD:SW_MEC_5GSH9, B.Cu at (-32.6, 11.0)
- added U4: XC6206P332MR, Package_TO_SOT_SMD:SOT-23_Handsoldering, B.Cu at (-57.8, 4.90)
- added U5: SGM2007-3.3XN5/TR, Package_TO_SOT_SMD:SOT-23-5_HandSoldering, B.Cu at (125.5, 154.2)
- C11, C12, C13, C14, C15, C16, C17, C18, C19, C20, C21, C22, C23, C24, C25: value 100nF -> 100n
- C26, Q1, R10, R12, R13, R15, R16, R18, R20, R23, R24, R25, R27, R32, R37, R44, R45, R51, R52, R54, R56, R58, R59, R60, R62, R65, R70, R73, R76, R77, R78, R79, R80, R81, R83, R85: moved to B.Cu
- C27: footprint Capacitor_SMD:C_0402_1005Metric -> Capacitor_SMD:C_0402_1005Metric_Pad0.74x0.62mm_HandSolder; moved to B.Cu
- D100, D101, D86, D87, D88, D89, D90, D91, D92, D93, D94, D95, D96, D97, D98, D99: value SK6812MINI-E -> WS2812C-2020; footprint LED_SMD:LED_SK6812MINI_PLCC4_3.5x3.5mm_P1.75mm -> acheron_Components:LED_WS2812_2020
- R2: value 100R -> 680R; moved to B.Cu
- R3: value 1k -> 680R; moved to B.Cu
- R4: value 330 -> 680R; moved to B.Cu
- R5: value 10k -> 680R; moved to B.Cu
- R6, R7: value 5.1k -> 680R
- R87: value 680R -> 5.1R; moved to B.Cu
- R88, R89, R90, R91, R92: value 680R -> 5.1R
- SWP1: value SW_Push -> SW_Push_RST; moved to B.Cu
- U2: value USBLC6-2SC6 -> STM32F072C8Tx; footprint acheron_Components:SOT-23-6 -> Package_QFP:LQFP-48_7x7mm_P0.5mm
- U3: value 74LVC1G125 -> USBLC6-2SC6; footprint Package_TO_SOT_SMD:SOT-23-5_HandSoldering -> Package_TO_SOT_SMD:SOT-23-6_Handsoldering; moved to B.Cu
- moved R63 252.7 mm to (209.7, 43.2)
- moved R41 181.7 mm to (133.5, 43.2)
- moved R51 179.9 mm to (171.5, 43.2), turned to 180 degrees
- moved R25 164.5 mm to (76.2, 43.2), turned to 180 degrees
- moved R57 160.3 mm to (190.5, 43.2)
- moved R86 149.9 mm to (285.7, 43.2)
- moved R20 147.1 mm to (57.2, 43.2), turned to 180 degrees
- moved R30 144.3 mm to (95.2, 43.2)
- moved R18 142.0 mm to (165.9, 161.4), turned to 180 degrees
- moved R15 141.5 mm to (24.2, 178.0), turned to 180 degrees
- moved R37 141.5 mm to (24.2, 171.4), turned to 180 degrees
- moved R52 141.5 mm to (24.2, 174.7), turned to 180 degrees
- moved R58 141.5 mm to (24.2, 168.2), turned to 180 degrees
- moved R2 140.9 mm to (-0.01, 43.2), turned to 180 degrees
- moved SWP1 136.3 mm to (163.0, 175.1), turned to 180 degrees
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Connections:
- C10 pad 1: GND -> Net-(C10-Pad1)
- C10 pad 2: +5V -> GND
- C11 pad 1: unconnected-(C11-Pad1) -> Net-(C11-Pad1)
- C12 pad 1: VCC -> Net-(C12-Pad1)
- C12 pad 2: unconnected-(C12-Pad2) -> GND
- C13 pad 2: unconnected-(C13-Pad2) -> GND
- C14 pad 2: Net-(C14-Pad2) -> GND
- C15 pad 2: Net-(C15-Pad2) -> GND
- C16 pad 1: Net-(C14-Pad1) -> Net-(C16-Pad1)
- C16 pad 2: Net-(C16-Pad2) -> GND
- C17 pad 1: Net-(C15-Pad1) -> Net-(C17-Pad1)
- C17 pad 2: Net-(C17-Pad2) -> GND
- C18 pad 2: Net-(C18-Pad2) -> GND
- C19 pad 2: Net-(C19-Pad2) -> GND
- C20 pad 1: unconnected-(C20-Pad1) -> Net-(C20-Pad1)
- C20 pad 2: Net-(C20-Pad2) -> GND
- C21 pad 2: Net-(C21-Pad2) -> GND
- C22 pad 2: Net-(C22-Pad2) -> GND
- C23 pad 2: Net-(C23-Pad2) -> GND
- C24 pad 1: unconnected-(C24-Pad1) -> Net-(C24-Pad1)
- C24 pad 2: Net-(C24-Pad2) -> GND
- C25 pad 2: Net-(C25-Pad2) -> GND
- C26 pad 1: unconnected-(C26-Pad1) -> +3V3
- C26 pad 2: Net-(C24-Pad2) -> GND
- C27 pad 1: unconnected-(C27-Pad1) -> RST
- C27 pad 2: Net-(C25-Pad2) -> GND
- D100 pad 1: unconnected-(D100-Pad1) -> Net-(D100-Pad1)
- D100 pad 2: unconnected-(D100-Pad2) -> GND
- D100 pad 3: Net-(C24-Pad2) -> Net-(D100-Pad3)
- D100 pad 4: unconnected-(D100-Pad4) -> Net-(C24-Pad1)
- D101 pad 1: Net-(C25-Pad1) -> Net-(D101-Pad1)
- D101 pad 2: unconnected-(D101-Pad2) -> GND
- D101 pad 3: Net-(C25-Pad2) -> Net-(D101-Pad3)
- D101 pad 4: unconnected-(D101-Pad4) -> Net-(C25-Pad1)
- D86 pad 1: VCC -> Net-(D86-Pad1)
- D86 pad 2: Net-(D86-Pad2) -> GND
- D86 pad 3: GND -> Net-(D100-Pad1)
- D86 pad 4: Net-(D86-Pad4) -> Net-(C10-Pad1)
- D87 pad 1: Net-(C13-Pad1) -> unconnected-(D87-Pad1)
- D87 pad 2: Net-(D87-Pad2) -> GND
- D87 pad 3: unconnected-(D87-Pad3) -> Net-(D101-Pad1)
- D87 pad 4: unconnected-(D87-Pad4) -> Net-(C11-Pad1)
- D88 pad 1: VCC -> Net-(D88-Pad1)
- D88 pad 2: Net-(D88-Pad2) -> GND
- D88 pad 3: Net-(C14-Pad2) -> UGLED
- D88 pad 4: Net-(D86-Pad2) -> Net-(C12-Pad1)
- D89 pad 1: Net-(C13-Pad1) -> Net-(D89-Pad1)
- D89 pad 2: Net-(D89-Pad2) -> GND
- D89 pad 3: unconnected-(D89-Pad3) -> Net-(D86-Pad1)
- D89 pad 4: Net-(D87-Pad2) -> Net-(C13-Pad1)
- D90 pad 1: Net-(C14-Pad1) -> Net-(D90-Pad1)
- D90 pad 2: Net-(D90-Pad2) -> GND
- D90 pad 3: Net-(C14-Pad2) -> Net-(D88-Pad1)
- D90 pad 4: Net-(D88-Pad2) -> Net-(C14-Pad1)
- D91 pad 1: Net-(C15-Pad1) -> Net-(D91-Pad1)
- D91 pad 2: Net-(D91-Pad2) -> GND
- D91 pad 3: Net-(C15-Pad2) -> Net-(D89-Pad1)
- D91 pad 4: Net-(D89-Pad2) -> Net-(C15-Pad1)
- D92 pad 1: Net-(C14-Pad1) -> Net-(D92-Pad1)
- D92 pad 2: unconnected-(D92-Pad2) -> GND
- D92 pad 3: Net-(C16-Pad2) -> Net-(D90-Pad1)
- D92 pad 4: Net-(D90-Pad2) -> Net-(C16-Pad1)
- D93 pad 1: Net-(C15-Pad1) -> Net-(D93-Pad1)
- D93 pad 2: unconnected-(D93-Pad2) -> GND
- D93 pad 3: Net-(C17-Pad2) -> Net-(D91-Pad1)
- D93 pad 4: Net-(D91-Pad2) -> Net-(C17-Pad1)
- D94 pad 1: Net-(C18-Pad1) -> Net-(D94-Pad1)
- D94 pad 2: Net-(D94-Pad2) -> GND
- D94 pad 3: Net-(C18-Pad2) -> Net-(D92-Pad1)
- D94 pad 4: unconnected-(D94-Pad4) -> Net-(C18-Pad1)
- D95 pad 1: Net-(C19-Pad1) -> Net-(D95-Pad1)
- D95 pad 2: Net-(D95-Pad2) -> GND
- D95 pad 3: Net-(C19-Pad2) -> Net-(D93-Pad1)
- D95 pad 4: unconnected-(D95-Pad4) -> Net-(C19-Pad1)
- D96 pad 1: unconnected-(D96-Pad1) -> Net-(D96-Pad1)
- D96 pad 2: Net-(D96-Pad2) -> GND
- D96 pad 3: Net-(C20-Pad2) -> Net-(D94-Pad1)
- D96 pad 4: Net-(D94-Pad2) -> Net-(C20-Pad1)
- D97 pad 1: Net-(C21-Pad1) -> Net-(D97-Pad1)
- D97 pad 2: Net-(D97-Pad2) -> GND
- D97 pad 3: Net-(C21-Pad2) -> Net-(D95-Pad1)
- D97 pad 4: Net-(D95-Pad2) -> Net-(C21-Pad1)
- D98 pad 1: Net-(C22-Pad1) -> Net-(D100-Pad3)
- D98 pad 2: unconnected-(D98-Pad2) -> GND
- D98 pad 3: Net-(C22-Pad2) -> Net-(D96-Pad1)
- D98 pad 4: Net-(D96-Pad2) -> Net-(C22-Pad1)
- D99 pad 1: Net-(C23-Pad1) -> Net-(D101-Pad3)
- D99 pad 2: unconnected-(D99-Pad2) -> GND
- D99 pad 3: Net-(C23-Pad2) -> Net-(D97-Pad1)
- D99 pad 4: Net-(D97-Pad2) -> Net-(C23-Pad1)
- MX82 pad 1: unconnected-(MX82-Pad1) -> col15
- R10 pad 1: Net-(MX3-Pad3) -> Net-(MX9-Pad3)
- R11 pad 1: Net-(MX4-Pad3) -> Net-(MX10-Pad3)
- R12 pad 1: Net-(MX5-Pad3) -> Net-(MX11-Pad3)
- R13 pad 1: Net-(MX6-Pad3) -> Net-(MX12-Pad3)
- R14 pad 1: Net-(MX7-Pad3) -> Net-(MX13-Pad3)
- R15 pad 1: Net-(MX8-Pad3) -> Net-(MX14-Pad3)
- R16 pad 1: Net-(MX9-Pad3) -> Net-(MX15-Pad3)
- R17 pad 1: Net-(MX10-Pad3) -> Net-(MX16-Pad3)
- R18 pad 1: Net-(MX11-Pad3) -> Net-(MX17-Pad3)
- R19 pad 1: Net-(MX12-Pad3) -> Net-(MX18-Pad3)
- R2 pad 1: LED_PWM -> Net-(MX1-Pad3)
- R2 pad 2: Net-(Q1-Pad1) -> LED-
- R20 pad 1: Net-(MX13-Pad3) -> Net-(MX19-Pad3)
- R21 pad 1: Net-(MX14-Pad3) -> Net-(MX20-Pad3)
- R22 pad 1: Net-(MX15-Pad3) -> Net-(MX21-Pad3)
- R23 pad 1: Net-(MX16-Pad3) -> Net-(MX22-Pad3)
- R24 pad 1: Net-(MX17-Pad3) -> Net-(MX23-Pad3)
- R25 pad 1: Net-(MX18-Pad3) -> Net-(MX24-Pad3)
- R26 pad 1: Net-(MX19-Pad3) -> Net-(MX25-Pad3)
- R27 pad 1: Net-(MX20-Pad3) -> Net-(MX26-Pad3)
- R28 pad 1: Net-(MX21-Pad3) -> Net-(MX27-Pad3)
- R29 pad 1: Net-(MX22-Pad3) -> Net-(MX28-Pad3)
- R3 pad 1: GND -> Net-(MX2-Pad3)
- R3 pad 2: Net-(R3-Pad2) -> LED-
- R30 pad 1: Net-(MX23-Pad3) -> Net-(MX29-Pad3)
- R31 pad 1: Net-(MX24-Pad3) -> Net-(MX30-Pad3)
- R32 pad 1: Net-(MX25-Pad3) -> Net-(MX31-Pad3)
- R33 pad 1: Net-(MX26-Pad3) -> Net-(MX32-Pad3)
- R34 pad 1: Net-(MX27-Pad3) -> Net-(MX33-Pad3)
- R35 pad 1: Net-(MX28-Pad3) -> Net-(MX34-Pad3)
- R36 pad 1: Net-(MX29-Pad3) -> Net-(MX35-Pad3)
- R37 pad 1: Net-(MX30-Pad3) -> Net-(MX36-Pad3)
- R38 pad 1: Net-(MX31-Pad3) -> Net-(MX37-Pad3)
- R39 pad 1: Net-(MX32-Pad3) -> Net-(MX38-Pad3)
- R4 pad 1: GND -> Net-(MX3-Pad3)
- R4 pad 2: Net-(R4-Pad2) -> LED-
- R40 pad 1: Net-(MX33-Pad3) -> Net-(MX39-Pad3)
- R41 pad 1: Net-(MX34-Pad3) -> Net-(MX40-Pad3)
- R42 pad 1: Net-(MX35-Pad3) -> Net-(MX41-Pad3)
- R43 pad 1: Net-(MX36-Pad3) -> Net-(MX42-Pad3)
- R44 pad 1: Net-(MX37-Pad3) -> Net-(MX43-Pad3)
- R45 pad 1: Net-(MX38-Pad3) -> Net-(MX44-Pad3)
- R46 pad 1: Net-(MX39-Pad3) -> Net-(MX45-Pad3)
- R47 pad 1: Net-(MX40-Pad3) -> Net-(MX46-Pad3)
- R48 pad 1: Net-(MX41-Pad3) -> Net-(MX47-Pad3)
- R49 pad 1: Net-(MX42-Pad3) -> Net-(MX48-Pad3)
- R5 pad 1: RST -> Net-(MX4-Pad3)
- R5 pad 2: +5V -> LED-
- R50 pad 1: Net-(MX43-Pad3) -> Net-(MX49-Pad3)
- R51 pad 1: Net-(MX44-Pad3) -> Net-(MX50-Pad3)
- R52 pad 1: Net-(MX45-Pad3) -> Net-(MX51-Pad3)
- R53 pad 1: Net-(MX46-Pad3) -> Net-(MX52-Pad3)
- R54 pad 1: Net-(MX47-Pad3) -> Net-(MX53-Pad3)
- R55 pad 1: Net-(MX48-Pad3) -> Net-(MX54-Pad3)
- R56 pad 1: Net-(MX49-Pad3) -> Net-(MX55-Pad3)
- R57 pad 1: Net-(MX50-Pad3) -> Net-(MX56-Pad3)
- R58 pad 1: Net-(MX51-Pad3) -> Net-(MX57-Pad3)
- R59 pad 1: Net-(MX52-Pad3) -> Net-(MX58-Pad3)
- R6 pad 1: GND -> Net-(MX5-Pad3)
- R6 pad 2: Net-(J1-PadB5) -> LED-
- R60 pad 1: Net-(MX53-Pad3) -> Net-(MX59-Pad3)
- R61 pad 1: Net-(MX54-Pad3) -> Net-(MX60-Pad3)
- R62 pad 1: Net-(MX55-Pad3) -> Net-(MX61-Pad3)
- R63 pad 1: Net-(MX56-Pad3) -> Net-(MX62-Pad3)
- R64 pad 1: Net-(MX57-Pad3) -> Net-(MX63-Pad3)
- R65 pad 1: Net-(MX58-Pad3) -> Net-(MX64-Pad3)
- R66 pad 1: Net-(MX59-Pad3) -> Net-(MX65-Pad3)
- R67 pad 1: Net-(MX60-Pad3) -> Net-(MX66-Pad3)
- R68 pad 1: Net-(MX61-Pad3) -> Net-(MX67-Pad3)
- R69 pad 1: Net-(MX62-Pad3) -> Net-(MX68-Pad3)
- R7 pad 1: GND -> Net-(MX6-Pad3)
- R7 pad 2: Net-(J1-PadA5) -> LED-
- R70 pad 1: Net-(MX63-Pad3) -> Net-(MX69-Pad3)
- R71 pad 1: Net-(MX64-Pad3) -> Net-(MX70-Pad3)
- R72 pad 1: Net-(MX65-Pad3) -> Net-(MX71-Pad3)
- R73 pad 1: Net-(MX66-Pad3) -> Net-(MX72-Pad3)
- R74 pad 1: Net-(MX67-Pad3) -> Net-(MX73-Pad3)
- R75 pad 1: Net-(MX68-Pad3) -> Net-(MX74-Pad3)
- R76 pad 1: Net-(MX69-Pad3) -> Net-(MX75-Pad3)
- R77 pad 1: Net-(MX70-Pad3) -> Net-(MX76-Pad3)
- R78 pad 1: Net-(MX71-Pad3) -> Net-(MX77-Pad3)
- R79 pad 1: Net-(MX72-Pad3) -> Net-(MX78-Pad3)
- R8 pad 1: Net-(MX1-Pad3) -> Net-(MX7-Pad3)
- R80 pad 1: Net-(MX73-Pad3) -> Net-(MX79-Pad3)
- R81 pad 1: Net-(MX74-Pad3) -> Net-(MX80-Pad3)
- R82 pad 1: Net-(MX75-Pad3) -> Net-(MX81-Pad3)
- R83 pad 1: Net-(MX76-Pad3) -> Net-(MX82-Pad3)
- R84 pad 1: Net-(MX77-Pad3) -> Net-(MX83-Pad3)
- R85 pad 1: Net-(MX78-Pad3) -> Net-(MX84-Pad3)
- R86 pad 1: Net-(MX79-Pad3) -> Net-(MX85-Pad3)
- R87 pad 1: Net-(MX80-Pad3) -> Net-(C10-Pad1)
- R87 pad 2: LED- -> 5V
- R88 pad 1: Net-(MX81-Pad3) -> Net-(C11-Pad1)
- R88 pad 2: LED- -> 5V
- R89 pad 1: Net-(MX82-Pad3) -> Net-(C12-Pad1)
- R89 pad 2: LED- -> 5V
- R9 pad 1: Net-(MX2-Pad3) -> Net-(MX8-Pad3)
- R90 pad 1: Net-(MX83-Pad3) -> Net-(C13-Pad1)
- R90 pad 2: LED- -> 5V
- R91 pad 1: Net-(MX84-Pad3) -> Net-(C14-Pad1)
- R91 pad 2: LED- -> 5V
- R92 pad 1: Net-(MX85-Pad3) -> Net-(C15-Pad1)
- R92 pad 2: LED- -> 5V
- SWP1 pad 1: Net-(R4-Pad2) -> Net-(R103-Pad2)
- U2 pad 1: D+ -> +3V3
- U2 pad 2: GND -> col6
- U2 pad 3: D- -> unconnected-(U2-Pad3)
- U2 pad 4: DBUS- -> unconnected-(U2-Pad4)
- U2 pad 5: VBUS -> col11
- U2 pad 6: DBUS+ -> col12
- U3 pad 1: GND -> D+
- U3 pad 2: UGLED -> GND
- U3 pad 3: GND -> D-
- U3 pad 4: Net-(D86-Pad4) -> DBUS-
- U3 pad 5: VCC -> VOUT
Routing:
- net +5V: track 358.6 -> 0.00 mm, vias 6 -> 0
- net GND: track 298.2 -> 0.00 mm, vias 4 -> 0
- net D-: track 204.8 -> 0.00 mm
- net D+: track 203.7 -> 0.00 mm
- net row1: track 309.0 -> 400.8 mm, vias 0 -> 2
- net VBUS: track 13.8 -> 0.00 mm, vias 3 -> 0
- net DBUS+: track 11.2 -> 0.00 mm, vias 2 -> 0
- net DBUS-: track 10.6 -> 0.00 mm, vias 2 -> 0
- net Net-(D1-Pad2): track 10.6 -> 0.00 mm
- net Net-(D7-Pad2): track 6.95 -> 0.00 mm
- net Net-(C2-Pad2): track 6.94 -> 0.00 mm
- net Net-(C1-Pad2): track 6.68 -> 0.00 mm
- net Net-(D19-Pad2): track 7.66 -> 2.89 mm
- net Net-(D45-Pad2): track 7.78 -> 3.06 mm
- net Net-(D50-Pad2): track 7.30 -> 2.79 mm
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
Commit message: added components on board and began routing
Parts:
- removed C35, C36, C37, C38: 100nF, Capacitor_SMD:C_0402_1005Metric
- removed C39, C41: 4.7uF, Capacitor_SMD:C_0402_1005Metric
- removed C40, C43: 1u, Capacitor_SMD:C_0805_2012Metric
- removed C42: 10n, Capacitor_SMD:C_0402_1005Metric
- removed F2: 500m, Fuse:Fuse_1206_3216Metric
- removed J2: USB_C_Receptacle_USB2.0, Connector_USB:USB_C_Receptacle_HRO_TYPE-C-31-M-12
- removed R102: 5.1R, Resistor_SMD:R_0402_1005Metric
- removed R103: 330, Resistor_SMD:R_0402_1005Metric
- removed R111: 5.1k, Resistor_SMD:R_0402_1005Metric
- removed R112: 100k, Resistor_SMD:R_0805_2012Metric
- removed U5: SGM2007-3.3XN5/TR, Package_TO_SOT_SMD:SOT-23-5_HandSoldering
- added C1: 100n, Capacitor_SMD:C_0402_1005Metric, B.Cu at (-73.3, 54.2)
- added C2: 100n, Capacitor_SMD:C_0402_1005Metric, B.Cu at (-76.2, 52.3)
- added C3: 100n, Capacitor_SMD:C_0402_1005Metric, B.Cu at (-70.5, 58.2)
- added C4: 100n, Capacitor_SMD:C_0402_1005Metric, B.Cu at (-76.2, 54.2)
- added C5: 100n, Capacitor_SMD:C_0402_1005Metric, B.Cu at (-70.5, 56.2)
- added C6: 100n, Capacitor_SMD:C_0402_1005Metric, B.Cu at (-73.3, 56.2)
- added C7: 100n, Capacitor_SMD:C_0402_1005Metric, B.Cu at (-70.5, 52.3)
- added C8: 100n, Capacitor_SMD:C_0402_1005Metric, B.Cu at (-73.3, 52.3)
- added C9: 100n, Capacitor_SMD:C_0402_1005Metric, B.Cu at (-70.5, 54.2)
- added FB1: GZ2012D601TF, Inductor_SMD:L_0805_2012Metric, B.Cu at (9.25, 34.3)
- added J1: TYPE-C-31-M12, acheron_Connectors:TYPE-C-31-M-12, B.Cu at (13.8, 32.2)
- added R1: 680R, Resistor_SMD:R_0402_1005Metric, B.Cu at (0.00, 43.2)
- added U1: STM32F072C8Tx, Package_QFP:LQFP-48_7x7mm_P0.5mm, B.Cu at (21.0, 75.0)
- C17, C24: value 100n -> 100nF
- C18: value 100n -> 100nF; footprint Capacitor_SMD:C_0402_1005Metric -> Capacitor_SMD:C_0402_1005Metric_Pad0.74x0.62mm_HandSolder
- C19, C20: value 100n -> 100uF; footprint Capacitor_SMD:C_0402_1005Metric -> Capacitor_Tantalum_SMD:CP_EIA-3528-21_Kemet-B
- C21: value 100n -> 10uF; footprint Capacitor_SMD:C_0402_1005Metric -> Capacitor_Tantalum_SMD:CP_EIA-3216-18_Kemet-A
- C22, C25: value 100n -> 1uF
- C23: value 100n -> 4.7uF
- C27: footprint Capacitor_SMD:C_0402_1005Metric_Pad0.74x0.62mm_HandSolder -> Capacitor_SMD:C_0402_1005Metric
- C28, C29: value 100uF -> 100nF; footprint Capacitor_Tantalum_SMD:CP_EIA-3528-21_Kemet-B -> Capacitor_SMD:C_0402_1005Metric
- C30: value 10uF -> 4.7uF; footprint Capacitor_Tantalum_SMD:CP_EIA-3216-18_Kemet-A -> Capacitor_SMD:C_0402_1005Metric
- C31, C34: value 1uF -> 1u; footprint Capacitor_SMD:C_0402_1005Metric -> Capacitor_SMD:C_0805_2012Metric
- C33: value 100nF -> 10n
- F1: footprint Fuse:Fuse_1206_3216Metric -> Fuse:Fuse_1206_3216Metric_Pad1.42x1.75mm_HandSolder
- R104, R105: value 10k -> 5.1k
- R106: value 100R -> 10k
- R107: value 10k -> 100R
- R108: value 0 -> 10k
- R110: value 5.1k -> 100k
- R86: value 680R -> 5.1R
- U2: value STM32F072C8Tx -> XC6206P332MR; footprint Package_QFP:LQFP-48_7x7mm_P0.5mm -> Package_TO_SOT_SMD:SOT-23_Handsoldering
- U4: value XC6206P332MR -> SGM2007-3.3XN5/TR; footprint Package_TO_SOT_SMD:SOT-23_Handsoldering -> Package_TO_SOT_SMD:SOT-23-5_HandSoldering
- moved D82 342.1 mm to (288.1, 90.2), turned to 0 degrees
- moved R84 334.5 mm to (285.7, 138.5)
- moved R19 305.0 mm to (57.0, 43.2)
- moved D72 296.3 mm to (242.8, 109.2), turned to 0 degrees
- moved D80 291.4 mm to (249.0, 60.0)
- moved D8 290.2 mm to (65.0, 93.0)
- moved D9 290.2 mm to (71.0, 98.0)
- moved R72 288.6 mm to (240.7, 119.5)
- moved R85 286.0 mm to (285.7, 43.2)
- moved R71 285.9 mm to (243.0, 100.2)
- moved D57 284.6 mm to (242.0, 55.0)
- moved D61 272.0 mm to (212.0, 128.2), turned to 0 degrees
- moved D20 269.6 mm to (65.0, 98.0)
- moved D66 265.8 mm to (216.5, 109.2), turned to 0 degrees
- moved R67 265.4 mm to (228.5, 138.5)
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Connections:
- C17 pad 1: Net-(C17-Pad1) -> +3V3
- C18 pad 1: Net-(C18-Pad1) -> RST
- C19 pad 1: Net-(C19-Pad1) -> +5V
- C20 pad 1: Net-(C20-Pad1) -> +5V
- C21 pad 1: Net-(C21-Pad1) -> +5V
- C22 pad 1: Net-(C22-Pad1) -> +5V
- C23 pad 1: Net-(C23-Pad1) -> +5V
- C24 pad 1: Net-(C24-Pad1) -> BOOT
- C25 pad 1: Net-(C25-Pad1) -> +3V3
- C27 pad 1: RST -> +3V3
- C28 pad 1: +5V -> +3V3
- C29 pad 1: +5V -> +3V3
- C30 pad 1: +5V -> +3V3
- C31 pad 1: +5V -> 5V
- C32 pad 1: +5V -> +3V3
- C33 pad 1: BOOT -> GND
- C33 pad 2: GND -> Net-(C33-Pad2)
- C34 pad 1: +3V3 -> GND
- C34 pad 2: GND -> 3V3
- D100 pad 4: Net-(C24-Pad1) -> Net-(C15-Pad1)
- D101 pad 4: Net-(C25-Pad1) -> Net-(C16-Pad1)
- D102 pad 1: 5V -> 3V3
- D102 pad 2: 3V3 -> 5V
- D86 pad 4: Net-(C10-Pad1) -> Net-(C1-Pad1)
- D87 pad 4: Net-(C11-Pad1) -> Net-(C2-Pad1)
- D88 pad 4: Net-(C12-Pad1) -> Net-(C3-Pad1)
- D89 pad 4: Net-(C13-Pad1) -> Net-(C4-Pad1)
- D90 pad 4: Net-(C14-Pad1) -> Net-(C5-Pad1)
- D91 pad 4: Net-(C15-Pad1) -> Net-(C6-Pad1)
- D92 pad 4: Net-(C16-Pad1) -> Net-(C7-Pad1)
- D93 pad 4: Net-(C17-Pad1) -> Net-(C8-Pad1)
- D94 pad 4: Net-(C18-Pad1) -> Net-(C9-Pad1)
- D95 pad 4: Net-(C19-Pad1) -> unconnected-(D95-Pad4)
- D96 pad 4: Net-(C20-Pad1) -> Net-(C11-Pad1)
- D97 pad 4: Net-(C21-Pad1) -> Net-(C12-Pad1)
- D98 pad 4: Net-(C22-Pad1) -> Net-(C13-Pad1)
- D99 pad 4: Net-(C23-Pad1) -> Net-(C14-Pad1)
- R10 pad 1: Net-(MX9-Pad3) -> Net-(MX10-Pad3)
- R100 pad 1: Net-(C23-Pad1) -> Net-(C15-Pad1)
- R101 pad 1: Net-(C24-Pad1) -> Net-(C16-Pad1)
- R104 pad 1: RST -> GND
- R104 pad 2: +5V -> Net-(J1-PadA5)
- R105 pad 1: LED_PWM -> Net-(J1-PadB5)
- R106 pad 2: Net-(Q1-Pad1) -> GND
- R107 pad 1: BOOT -> LED_PWM
- R107 pad 2: GND -> Net-(Q1-Pad1)
- R108 pad 1: Net-(J2-PadA1) -> BOOT
- R11 pad 1: Net-(MX10-Pad3) -> Net-(MX11-Pad3)
- R110 pad 1: GNDPWR -> GND
- R110 pad 2: Net-(J2-PadA5) -> 3V3
- R12 pad 1: Net-(MX11-Pad3) -> Net-(MX12-Pad3)
- R13 pad 1: Net-(MX12-Pad3) -> Net-(MX13-Pad3)
- R14 pad 1: Net-(MX13-Pad3) -> Net-(MX14-Pad3)
- R15 pad 1: Net-(MX14-Pad3) -> Net-(MX15-Pad3)
- R16 pad 1: Net-(MX15-Pad3) -> Net-(MX16-Pad3)
- R17 pad 1: Net-(MX16-Pad3) -> Net-(MX17-Pad3)
- R18 pad 1: Net-(MX17-Pad3) -> Net-(MX18-Pad3)
- R19 pad 1: Net-(MX18-Pad3) -> Net-(MX19-Pad3)
- R2 pad 1: Net-(MX1-Pad3) -> Net-(MX2-Pad3)
- R20 pad 1: Net-(MX19-Pad3) -> Net-(MX20-Pad3)
- R21 pad 1: Net-(MX20-Pad3) -> Net-(MX21-Pad3)
- R22 pad 1: Net-(MX21-Pad3) -> Net-(MX22-Pad3)
- R23 pad 1: Net-(MX22-Pad3) -> Net-(MX23-Pad3)
- R24 pad 1: Net-(MX23-Pad3) -> Net-(MX24-Pad3)
- R25 pad 1: Net-(MX24-Pad3) -> Net-(MX25-Pad3)
- R26 pad 1: Net-(MX25-Pad3) -> Net-(MX26-Pad3)
- R27 pad 1: Net-(MX26-Pad3) -> Net-(MX27-Pad3)
- R28 pad 1: Net-(MX27-Pad3) -> Net-(MX28-Pad3)
- R29 pad 1: Net-(MX28-Pad3) -> Net-(MX29-Pad3)
- R3 pad 1: Net-(MX2-Pad3) -> Net-(MX3-Pad3)
- R30 pad 1: Net-(MX29-Pad3) -> Net-(MX30-Pad3)
- R31 pad 1: Net-(MX30-Pad3) -> Net-(MX31-Pad3)
- R32 pad 1: Net-(MX31-Pad3) -> Net-(MX32-Pad3)
- R33 pad 1: Net-(MX32-Pad3) -> Net-(MX33-Pad3)
- R34 pad 1: Net-(MX33-Pad3) -> Net-(MX34-Pad3)
- R35 pad 1: Net-(MX34-Pad3) -> Net-(MX35-Pad3)
- R36 pad 1: Net-(MX35-Pad3) -> Net-(MX36-Pad3)
- R37 pad 1: Net-(MX36-Pad3) -> Net-(MX37-Pad3)
- R38 pad 1: Net-(MX37-Pad3) -> Net-(MX38-Pad3)
- R39 pad 1: Net-(MX38-Pad3) -> Net-(MX39-Pad3)
- R4 pad 1: Net-(MX3-Pad3) -> Net-(MX4-Pad3)
- R40 pad 1: Net-(MX39-Pad3) -> Net-(MX40-Pad3)
- R41 pad 1: Net-(MX40-Pad3) -> Net-(MX41-Pad3)
- R42 pad 1: Net-(MX41-Pad3) -> Net-(MX42-Pad3)
- R43 pad 1: Net-(MX42-Pad3) -> Net-(MX43-Pad3)
- R44 pad 1: Net-(MX43-Pad3) -> Net-(MX44-Pad3)
- R45 pad 1: Net-(MX44-Pad3) -> Net-(MX45-Pad3)
- R46 pad 1: Net-(MX45-Pad3) -> Net-(MX46-Pad3)
- R47 pad 1: Net-(MX46-Pad3) -> Net-(MX47-Pad3)
- R48 pad 1: Net-(MX47-Pad3) -> Net-(MX48-Pad3)
- R49 pad 1: Net-(MX48-Pad3) -> Net-(MX49-Pad3)
- R5 pad 1: Net-(MX4-Pad3) -> Net-(MX5-Pad3)
- R50 pad 1: Net-(MX49-Pad3) -> Net-(MX50-Pad3)
- R51 pad 1: Net-(MX50-Pad3) -> Net-(MX51-Pad3)
- R52 pad 1: Net-(MX51-Pad3) -> Net-(MX52-Pad3)
- R53 pad 1: Net-(MX52-Pad3) -> Net-(MX53-Pad3)
- R54 pad 1: Net-(MX53-Pad3) -> Net-(MX54-Pad3)
- R55 pad 1: Net-(MX54-Pad3) -> Net-(MX55-Pad3)
- R56 pad 1: Net-(MX55-Pad3) -> Net-(MX56-Pad3)
- R57 pad 1: Net-(MX56-Pad3) -> Net-(MX57-Pad3)
- R58 pad 1: Net-(MX57-Pad3) -> Net-(MX58-Pad3)
- R59 pad 1: Net-(MX58-Pad3) -> Net-(MX59-Pad3)
- R6 pad 1: Net-(MX5-Pad3) -> Net-(MX6-Pad3)
- R60 pad 1: Net-(MX59-Pad3) -> Net-(MX60-Pad3)
- R61 pad 1: Net-(MX60-Pad3) -> Net-(MX61-Pad3)
- R62 pad 1: Net-(MX61-Pad3) -> Net-(MX62-Pad3)
- R63 pad 1: Net-(MX62-Pad3) -> Net-(MX63-Pad3)
- R64 pad 1: Net-(MX63-Pad3) -> Net-(MX64-Pad3)
- R65 pad 1: Net-(MX64-Pad3) -> Net-(MX65-Pad3)
- R66 pad 1: Net-(MX65-Pad3) -> Net-(MX66-Pad3)
- R67 pad 1: Net-(MX66-Pad3) -> Net-(MX67-Pad3)
- R68 pad 1: Net-(MX67-Pad3) -> Net-(MX68-Pad3)
- R69 pad 1: Net-(MX68-Pad3) -> Net-(MX69-Pad3)
- R7 pad 1: Net-(MX6-Pad3) -> Net-(MX7-Pad3)
- R70 pad 1: Net-(MX69-Pad3) -> Net-(MX70-Pad3)
- R71 pad 1: Net-(MX70-Pad3) -> Net-(MX71-Pad3)
- R72 pad 1: Net-(MX71-Pad3) -> Net-(MX72-Pad3)
- R73 pad 1: Net-(MX72-Pad3) -> Net-(MX73-Pad3)
- R74 pad 1: Net-(MX73-Pad3) -> Net-(MX74-Pad3)
- R75 pad 1: Net-(MX74-Pad3) -> Net-(MX75-Pad3)
- R76 pad 1: Net-(MX75-Pad3) -> Net-(MX76-Pad3)
- R77 pad 1: Net-(MX76-Pad3) -> Net-(MX77-Pad3)
- R78 pad 1: Net-(MX77-Pad3) -> Net-(MX78-Pad3)
- R79 pad 1: Net-(MX78-Pad3) -> Net-(MX79-Pad3)
- R8 pad 1: Net-(MX7-Pad3) -> Net-(MX8-Pad3)
- R80 pad 1: Net-(MX79-Pad3) -> Net-(MX80-Pad3)
- R81 pad 1: Net-(MX80-Pad3) -> Net-(MX81-Pad3)
- R82 pad 1: Net-(MX81-Pad3) -> Net-(MX82-Pad3)
- R83 pad 1: Net-(MX82-Pad3) -> Net-(MX83-Pad3)
- R84 pad 1: Net-(MX83-Pad3) -> Net-(MX84-Pad3)
- R85 pad 1: Net-(MX84-Pad3) -> Net-(MX85-Pad3)
- R86 pad 1: Net-(MX85-Pad3) -> Net-(C1-Pad1)
- R86 pad 2: LED- -> 5V
- R87 pad 1: Net-(C10-Pad1) -> Net-(C2-Pad1)
- R88 pad 1: Net-(C11-Pad1) -> Net-(C3-Pad1)
- R89 pad 1: Net-(C12-Pad1) -> Net-(C4-Pad1)
- R9 pad 1: Net-(MX8-Pad3) -> Net-(MX9-Pad3)
- R90 pad 1: Net-(C13-Pad1) -> Net-(C5-Pad1)
- R91 pad 1: Net-(C14-Pad1) -> Net-(C6-Pad1)
- R92 pad 1: Net-(C15-Pad1) -> Net-(C7-Pad1)
- R93 pad 1: Net-(C16-Pad1) -> Net-(C8-Pad1)
- R94 pad 1: Net-(C17-Pad1) -> Net-(C9-Pad1)
- R95 pad 1: Net-(C18-Pad1) -> Net-(C10-Pad1)
- R96 pad 1: Net-(C19-Pad1) -> Net-(C11-Pad1)
- R97 pad 1: Net-(C20-Pad1) -> Net-(C12-Pad1)
- R98 pad 1: Net-(C21-Pad1) -> Net-(C13-Pad1)
- R99 pad 1: Net-(C22-Pad1) -> Net-(C14-Pad1)
- SWP1 pad 1: Net-(R103-Pad2) -> GND
- U2 pad 1: +3V3 -> GND
- U2 pad 2: col6 -> +3V3
- U2 pad 3: unconnected-(U2-Pad3) -> +5V
- U3 pad 5: VOUT -> VBUS
- U4 pad 1: GND -> 5V
- U4 pad 2: +3V3 -> GND
- U4 pad 3: +5V -> 5V
Routing:
- net LED-: track 0.00 -> 973.7 mm, vias 0 -> 6
- net VBUS: track 0.00 -> 174.4 mm, vias 0 -> 5
- net row1: track 400.8 -> 306.7 mm
- net +3V3: track 0.00 -> 58.2 mm, vias 0 -> 4
- net Net-(Q1-Pad1): track 0.00 -> 35.2 mm, vias 0 -> 2
- net GND: track 0.00 -> 34.1 mm, vias 0 -> 2
- net D+: track 0.00 -> 30.4 mm
- net D-: track 0.00 -> 30.4 mm
- net 5V: track 0.00 -> 28.2 mm, vias 0 -> 1
- net GNDPWR: track 0.00 -> 19.6 mm
- net LED_PWM: track 0.00 -> 16.8 mm
- net DBUS+: track 0.00 -> 14.2 mm, vias 0 -> 2
- net DBUS-: track 0.00 -> 13.6 mm, vias 0 -> 2
- net 3V3: track 0.00 -> 13.3 mm, vias 0 -> 1
- net col5: track 0.00 -> 7.26 mm, vias 0 -> 1
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Other:
- outline, holes or cut-outs redrawn

Commit message: Added some routes and finished to align components on switches
Parts:
- moved D63 134.0 mm to (211.8, 52.0), turned to 0 degrees
- moved D64 101.9 mm to (221.2, 71.0), turned to 0 degrees
- moved D81 93.2 mm to (288.0, 71.2), turned to 0 degrees
- moved D2 74.3 mm to (2.25, 52.0), turned to 0 degrees
- moved D4 68.7 mm to (9.50, 90.2), turned to 0 degrees
- moved D5 66.3 mm to (4.75, 109.0), turned to 0 degrees
- moved D11 60.0 mm to (26.2, 109.2), turned to 0 degrees
- moved D8 59.8 mm to (21.5, 52.0), turned to 0 degrees
- moved R18 59.7 mm to (50.8, 138.5)
- moved R12 59.4 mm to (26.5, 138.5)
- moved D3 57.0 mm to (7.00, 71.2), turned to 0 degrees
- moved D36 56.1 mm to (126.2, 71.2), turned to 0 degrees
- moved R87 55.0 mm to (80.2, 155.0)
- moved D57 49.5 mm to (192.6, 52.0), turned to 0 degrees
- moved D9 48.5 mm to (30.8, 71.0), turned to 0 degrees
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Routing:
- net LED-: track 973.7 -> 1347.8 mm
- net row3: track 0.00 -> 319.9 mm, vias 0 -> 3
- net row2: track 0.00 -> 309.3 mm, vias 0 -> 3
- net row4: track 0.00 -> 299.3 mm, vias 0 -> 3
- net row5: track 0.00 -> 65.0 mm, vias 0 -> 1
- net Net-(D12-Pad2): track 0.00 -> 3.31 mm
- net Net-(D57-Pad2): track 0.00 -> 3.26 mm
- net Net-(D58-Pad2): track 0.00 -> 3.23 mm
- net Net-(D17-Pad2): track 0.00 -> 3.21 mm
- net Net-(D54-Pad2): track 0.00 -> 3.21 mm
- net Net-(D9-Pad2): track 0.00 -> 3.21 mm
- net Net-(D64-Pad2): track 0.00 -> 3.21 mm
- net Net-(D76-Pad2): track 0.00 -> 3.21 mm
- net Net-(D46-Pad2): track 0.00 -> 3.20 mm
- net Net-(D75-Pad2): track 0.00 -> 3.19 mm
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
Commit message: routed all rows and backlight RGB
Routing:
- net LED-: track 1347.8 -> 1941.0 mm
- net row6: track 2.33 -> 300.2 mm, vias 1 -> 3
- net row5: track 65.0 -> 302.3 mm
