File: snk75/snk75.kicad_pcb (KiCad board)
At the start: 2 copper layers, 314.3 x 123.8 mm, 332 parts, among them J1 TYPE-C-31-M12, Q1 AO3400A, U1 STM32F072C8Tx, U3 USBLC6-2SC6, U4 SGM2007-3.3XN5/TR

Commit message: Nearly make all paths
Parts:
- removed C30: 4.7uF, Capacitor_SMD:C_0402_1005Metric
- removed C31, C34: 1u, Capacitor_SMD:C_0805_2012Metric
- removed C33: 10n, Capacitor_SMD:C_0402_1005Metric
- removed R109, R110: 100k, Resistor_SMD:R_0402_1005Metric
- removed U4: SGM2007-3.3XN5/TR, Package_TO_SOT_SMD:SOT-23-5_HandSoldering
- added C19: 100nF, Capacitor_SMD:C_0402_1005Metric, B.Cu at (95.0, 136.8)
- added C20: 1uF, Capacitor_SMD:C_0402_1005Metric, B.Cu at (11.8, 67.2)
- added C21: 1uF, Capacitor_SMD:C_0805_2012Metric, B.Cu at (72.2, 131.8)
- added C22: 10nF, Capacitor_SMD:C_0402_1005Metric, B.Cu at (17.0, 80.5)
- added C23: 100nF, Capacitor_SMD:C_0402_1005Metric, B.Cu at (25.0, 73.2)
- added R102: 5.1k, Resistor_SMD:R_0402_1005Metric, B.Cu at (11.5, 35.8)
- added R103: 5.1k, Resistor_SMD:R_0402_1005Metric, B.Cu at (16.2, 35.2)
- added U2: USBLC6-2SC6, Package_TO_SOT_SMD:SOT-23-6_Handsoldering, B.Cu at (14.0, 39.5)
- C1, C10, C11, C12, C13, C14, C15, C16, C2, C3, C4, C5, C6, C7, C8, C9: value 100n -> 100nF
- C25: value 1uF -> 10nF
- C27, C29: value 100nF -> 4.7uF
- C28: value 100nF -> 1uF; footprint Capacitor_SMD:C_0402_1005Metric -> Capacitor_SMD:C_0805_2012Metric
- D1, D10, D11, D12, D13, D14, D15, D16, D17, D18, D19, D2, D20, D21, D22, D23, D24, D25, D26, D27, D28, D29, D3, D30, D31, D32, D33, D34, D35, D36, D37, D38, D39, D4, D40, D41, D42, D43, D44, D45, D46, D47, D48, D49, D5, D50, D51, D52, D53, D54, D55, D56, D57, D58, D59, D6, D60, D61, D62, D63, D64, D65, D66, D67, D68, D69, D7, D70, D71, D72, D73, D74, D75, D76, D77, D78, D79, D8, D80, D81, D82, D83, D84, D85, D9: value 1N14148W -> 1N4148W
- R104: value 5.1k -> 10k
- R105: value 5.1k -> 100R
- R107: value 100R -> 100k
- R108: value 10k -> 100k
- SWP1, SWP2: footprint Button_Switch_SMD:SW_MEC_5GSH9 -> Button_Switch_SMD:SW_SPST_SKQG_WithStem
- U3: value USBLC6-2SC6 -> SGM2007-3.3XN5/TR; footprint Package_TO_SOT_SMD:SOT-23-6_Handsoldering -> Package_TO_SOT_SMD:SOT-23-5_HandSoldering
- moved C4 378.7 mm to (291.5, 145.0), turned to -90 degrees
- moved R100 374.5 mm to (293.0, 65.2), turned to 0 degrees
- moved C1 369.9 mm to (293.0, 105.2), turned to -90 degrees
- moved R98 364.2 mm to (288.8, 45.8), turned to 0 degrees
- moved C6 319.9 mm to (234.0, 145.0), turned to -90 degrees
- moved R96 305.0 mm to (231.5, 45.8), turned to 0 degrees
- moved R93 272.8 mm to (162.0, 143.5), turned to 90 degrees
- moved R94 254.3 mm to (174.8, 45.8), turned to 0 degrees
- moved C8 251.8 mm to (160.8, 145.0), turned to -90 degrees
- moved C9 244.3 mm to (173.8, 47.6), turned to -90 degrees
- moved R95 233.3 mm to (117.5, 143.8), turned to 90 degrees
- moved D99 231.9 mm to (6.75, 142.9)
- moved C14 227.5 mm to (7.68, 145.0), turned to -90 degrees
- moved R86 227.1 mm to (293.5, 103.5), turned to 0 degrees
- moved D101 226.0 mm to (-2.50, 104.8), turned to 90 degrees
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Connections:
- C24 pad 1: BOOT -> +3V3
- C25 pad 1: +3V3 -> GND
- C25 pad 2: GND -> Net-(C25-Pad2)
- C28 pad 1: +3V3 -> GND
- C28 pad 2: GND -> +3V3
- D102 pad 2: 5V -> +5V
- D95 pad 4: unconnected-(D95-Pad4) -> Net-(C10-Pad1)
- F1 pad 1: 5V -> +5V
- R100 pad 2: 5V -> +5V
- R101 pad 2: 5V -> +5V
- R104 pad 1: GND -> LED_PWM
- R104 pad 2: Net-(J1-PadA5) -> GND
- R105 pad 1: Net-(J1-PadB5) -> LED_PWM
- R105 pad 2: GND -> Net-(Q1-Pad1)
- R106 pad 1: LED_PWM -> BOOT
- R107 pad 1: LED_PWM -> +5V
- R107 pad 2: Net-(Q1-Pad1) -> GND
- R108 pad 1: BOOT -> GND
- R108 pad 2: GND -> +3V3
- R86 pad 2: 5V -> +5V
- R87 pad 2: 5V -> +5V
- R88 pad 2: 5V -> +5V
- R89 pad 2: 5V -> +5V
- R90 pad 2: 5V -> +5V
- R91 pad 2: 5V -> +5V
- R92 pad 2: 5V -> +5V
- R93 pad 2: 5V -> +5V
- R94 pad 2: 5V -> +5V
- R95 pad 2: 5V -> +5V
- R96 pad 2: 5V -> +5V
- R97 pad 2: 5V -> +5V
- R98 pad 2: 5V -> +5V
- R99 pad 2: 5V -> +5V
- U3 pad 1: D+ -> +5V
- U3 pad 3: D- -> +5V
- U3 pad 4: DBUS- -> Net-(C25-Pad2)
- U3 pad 5: VBUS -> +3V3
Routing:
- net +5V: track 0.00 -> 2333.8 mm, vias 0 -> 26
- net +3V3: track 36.9 -> 181.2 mm, vias 0 -> 11
- net Net-(D91-Pad1): track 0.00 -> 72.5 mm
- net Net-(D92-Pad1): track 0.00 -> 57.1 mm
- net Net-(D90-Pad1): track 0.00 -> 56.8 mm
- net Net-(D96-Pad1): track 0.00 -> 56.6 mm
- net Net-(D94-Pad1): track 0.00 -> 56.2 mm
- net Net-(D89-Pad1): track 0.00 -> 56.2 mm
- net Net-(D88-Pad1): track 0.00 -> 55.9 mm
- net Net-(D95-Pad1): track 0.00 -> 53.5 mm
- net Net-(D97-Pad1): track 0.00 -> 52.9 mm
- net UGLED: track 5.18 -> 51.4 mm, vias 1 -> 2
- net Net-(D93-Pad1): track 0.00 -> 43.2 mm
- net Net-(D101-Pad3): track 0.00 -> 41.4 mm
- net Net-(D86-Pad1): track 0.00 -> 40.9 mm
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- removed copper zone on B.Cu, net GND
- removed copper zone on F.Cu, net GND

Commit message: WIP: replacing backlight LEDs with RGB LEDs
Parts:
- removed R1: 680R, Resistor_SMD:R_0402_1005Metric
- MX1, MX10, MX11, MX13, MX14, MX15, MX16, MX17, MX19, MX2, MX20, MX21, MX22, MX23, MX24, MX25, MX26, MX27, MX28, MX29, MX30, MX31, MX32, MX33, MX34, MX35, MX36, MX37, MX38, MX40, MX41, MX42, MX43, MX44, MX45, MX46, MX47, MX48, MX49, MX50, MX51, MX52, MX53, MX54, MX55, MX56, MX57, MX58, MX59, MX60, MX61, MX62, MX63, MX64, MX65, MX66, MX67, MX68, MX69, MX7, MX70, MX71, MX73, MX74, MX77, MX78, MX79, MX8, MX80, MX81, MX82, MX83, MX84, MX85, MX9: footprint MX_Only:MXOnly-1U -> MX_Only:MXOnly-1U-NoLED
- MX12, MX18, MX5, MX6: footprint MX_Only:MXOnly-1.25U -> MX_Only:MXOnly-1.25U-NoLED
- MX3: footprint MX_Only:MXOnly-1.5U -> MX_Only:MXOnly-1.5U-NoLED
- MX39: footprint MX_Only:MXOnly-6.25U -> MX_Only:MXOnly-6.25U-NoLED
- MX4, MX72: footprint MX_Only:MXOnly-1.75U -> MX_Only:MXOnly-1.75U-NoLED
- MX75: footprint MX_Only:MXOnly-2U -> MX_Only:MXOnly-2U-NoLED
- MX76: footprint MX_Only:MXOnly-ISO -> MX_Only:MXOnly-ISO-NoLED
Routing:
- net LED-: track 1911.1 -> 1889.0 mm
- net +5V: track 2333.8 -> 2337.2 mm, vias 26 -> 23
- net col15: track 503.7 -> 500.7 mm
- net col14: track 483.4 -> 480.3 mm
- net col16: track 515.1 -> 512.0 mm
- net Net-(MX1-Pad3): track 2.69 -> 0.00 mm
